Commit message: versione provata su robot

File: locosim/robot_urdf/generated_urdf/ur5.urdf (robot description, URDF)
Before this commit: robot ur_robot, 30 links, 29 joints
Links:
- removed link hand_1_link2
- removed link hand_2_link2
- added link gripper_base_down, mass 1.0; collision mesh filename=package://gripper_description/meshes/gripper_base_down.stl scale=0.001 0.001 0.001; visual mesh filename=package://gripper_description/meshes/gripper_base_down.stl scale=0.001 0.001 0.001
- added link hand_3_link, mass 0.05; collision mesh filename=package://gripper_description/meshes/finger.stl scale=0.001 0.001 0.001; visual mesh filename=package://gripper_description/meshes/finger.stl scale=0.001 0.001 0.001
- link gripper_base: mass 0.168 -> None; geometry collision mesh filename=package://gripper_description/meshes/gripper_base_up.stl scale=0.001 0.001 0.001; visual mesh filename=package://gripper_description/meshes/gripper_base_up.stl scale=0.001 0.001 0.001
- link hand_1_link: mass 0.168 -> 0.05; geometry collision mesh filename=package://gripper_description/meshes/finger.stl scale=0.001 0.001 0.001; visual mesh filename=package://gripper_description/meshes/finger.stl scale=0.001 0.001 0.001
- link hand_2_link: mass 0.168 -> 0.05; geometry collision mesh filename=package://gripper_description/meshes/finger.stl scale=0.001 0.001 0.001; visual mesh filename=package://gripper_description/meshes/finger.stl scale=0.001 0.001 0.001
- link zed2_camera_center: geometry collision mesh filename=package://ur_description/sensors/zed2/ZED2.dae; visual mesh filename=package://ur_description/sensors/zed2/ZED2.dae
Joints:
- removed joint hand_1_joint2
- removed joint hand_2_joint2
- added joint flange: type fixed, parent gripper_base, child gripper_base_down, origin xyz=0 0 0.06 rpy=0 0 0
- added joint hand_3_joint: type revolute, parent gripper_base_down, child hand_3_link, origin xyz=-0.02598 0.015 0.05 rpy=-1.5707963267948966 0 -2.0943951023931953, axis 0 -1 0, limit lower=0 upper=3.14 effort=50 velocity=10.0
- joint gripper_robot_joint: origin xyz=0 0 0 rpy=0 0 1.57 -> xyz=0 0 0 rpy=0 0 3.14
- joint hand_1_joint: axis (none) -> 0 -1 0; limit (none) -> lower=0 upper=3.14 effort=50 velocity=10.0; origin xyz=0 -0.028 0.09 rpy= 0 0 0 -> xyz=0.0  -0.03 0.05 rpy=-1.5707963267948966 0 0; parent gripper_base -> gripper_base_down; type fixed -> revolute
- joint hand_2_joint: axis (none) -> 0 -1 0; limit (none) -> lower=0 upper=3.14 effort=50 velocity=10.0; origin xyz=0 0.028 0.09 rpy= 0 0 -3.141592653589793 -> xyz=0.02598 0.015 0.05 rpy=-1.5707963267948966 0 2.0943951023931953; parent gripper_base -> gripper_base_down; type fixed -> revolute
- joint zed_camera_fixed_joint: origin xyz=-0.9 0.065 -0.30 rpy=0. 0.523 0. -> xyz=-0.9 0.065 -0.3 rpy=0. 0.523 0.
