Commit message: grasping in simulazione abbastanza stabile, aggiunto controllo per altezza, diametro e posizionamento dei blocchi in base alla classe, modificata l'apertura massima del soft gripper

File: locosim/robot_descriptions/gripper_description/urdf/gripper.macro.xacro (robot description, xacro)
@@ -85,6 +85,6 @@
 		       <forces_angle_tolerance>100</forces_angle_tolerance>
 		       <update_rate>500</update_rate>
-		       <grip_count_threshold>4</grip_count_threshold>
-		       <max_grip_count>20</max_grip_count>
+		       <grip_count_threshold>3</grip_count_threshold>
+		       <max_grip_count>10</max_grip_count>
 		       <release_tolerance>0.005</release_tolerance>
 		       <disable_collisions_on_attach>true</disable_collisions_on_attach>

File: locosim/robot_descriptions/gripper_description/urdf/soft_finger.xacro (robot description, xacro)
@@ -16,5 +16,5 @@
 	    <axis xyz="1 0 0"/>
 	    <xacro:insert_block name="origin"/>
-	    <limit effort="50" velocity="10.0" lower="-0.5" upper="0.3" />
+	    <limit effort="50" velocity="10.0" lower="-1" upper="1" />
 	  </joint>
 	</xacro:if>

File: locosim/robot_descriptions/gripper_description/urdf/soft_gripper.macro.xacro (robot description, xacro)
@@ -14,5 +14,5 @@
 	    </visual>
 	    <collision>
-	        <origin rpy="0 0 0" xyz="0 0 -0.0095" />
+	        <origin rpy="0 0 0" xyz="0 0 0" />
 	    <geometry>
 		    <mesh filename="package://gripper_description/meshes/soft_gripper_base_down.stl"/>
@@ -59,6 +59,6 @@
 			   <gripper_link> hand_2_link </gripper_link>
 			</arm>
-		       <forces_angle_tolerance>100</forces_angle_tolerance>
-		       <update_rate>500</update_rate>
+		       <forces_angle_tolerance>91</forces_angle_tolerance>
+		       <update_rate>1000</update_rate>
 		       <grip_count_threshold>3</grip_count_threshold>
 		       <max_grip_count>10</max_grip_count>
