Commit message: per push dei commit precedenti

File: locosim/robot_descriptions/gripper_description/urdf/soft_finger.xacro (robot description, xacro)
@@ -58,7 +58,20 @@
 	</visual>
 	<collision>
-		<geometry>
-		  <mesh filename="package://gripper_description/meshes/soft_gripper_finger2.stl" />
-		</geometry>
+	  <geometry>
+	    <mesh filename="package://gripper_description/meshes/soft_gripper_finger2.stl" />
+	      <surface>
+	        <friction>
+	          <ode>
+	            <mu>10000000000</mu>
+	            <mu2>100000000000</mu2>
+	            <fdir1>0 0 1</fdir1>
+		  </ode>
+		</friction>
+		<contact>
+		  <poissons_ratio>0.5</poissons_ratio>
+		  <elastic_modulus>1e8</elastic_modulus>
+		</contact>
+		</surface>
+	      </geometry>
 	</collision>
 	<inertial>
@@ -76,25 +89,5 @@
 	 <gazebo reference="${name}_link">
 	    <collision name="${name}_link_collision">
-	      <surface>
-		<friction>
-		  <torsional>
-		    <coefficient>10.0</coefficient>
-		    <use_patch_radius>true</use_patch_radius>
-		    <patch_radius>0.05</patch_radius>
-		  </torsional>
-		</friction>
-		<contact>
-		  <poissons_ratio>0.5</poissons_ratio>
-		  <elastic_modulus>1e8</elastic_modulus>
-		</contact>
-	      </surface>
 	    </collision>
-	    <mu1>10</mu1>
-	    <mu2>10</mu2>
-	    <kp>1000000.0</kp>
-	    <kd>10.0</kd>
-	    <fdir1>0 0 1</fdir1>
-	    <minDepth>0.001</minDepth>
-		    <maxVel>0.0</maxVel>
 	    <maxContacts>1</maxContacts>
 	    <material>Gazebo/RedBright</material>

File: locosim/robot_descriptions/ur_description/urdf/ur5.urdf.xacro (robot description, xacro)
@@ -6,6 +6,7 @@
 <xacro:arg name="gripper"       default="true"/>
 <xacro:arg name="soft_gripper"  default="false" />
+<xacro:arg name="use_grasp_plugin" default="false" />
 <xacro:arg name="prefix" default=""/>
-<xacro:arg name="transmission_hw_interface" default="hardware_interface/EffortJointInterface"/>
+<xacro:arg name="transmission_hw_interface" default="hardware_interface/VelocityJointInterface"/>
 <xacro:arg name="joint_limit_params" default="$(find ur_description)/config/ur5e/joint_limits.yaml"/>
 <xacro:arg name="kinematics_params"  default="$(find ur_description)/config/ur5e/default_kinematics.yaml"/>
@@ -34,5 +35,5 @@
 	<xacro:soft_gripper
 	transmission_hw_interface="$(arg transmission_hw_interface)"
-	grasp_plugin=  "$(arg gripper)"
+	grasp_plugin=  "$(arg use_grasp_plugin)"
 	gripper_active="$(arg gripper)"/>
 </xacro:if>
@@ -41,5 +42,5 @@
 	<xacro:gripper
 		transmission_hw_interface="$(arg transmission_hw_interface)"
-		grasp_plugin=  "$(arg gripper)"
+		grasp_plugin=  "$(arg use_grasp_plugin)"
 		gripper_active="$(arg gripper)"/>
 </xacro:unless>
@@ -142,29 +143,5 @@
       <selfCollide>true</selfCollide>
     </gazebo>
-	<!-- fix me https://answers.gazebosim.org//question/15095/gazebo-contact-sensor-added-to-a-robot-link-in-urdf-file-is-not-working-as-expected/-->
-	<!--gazebo reference="$(arg prefix)wrist_3_link">
-		<kp>1000000.0</kp>
-		<kd>100.0</kd>
-		<mu1>1.0</mu1>
-		<mu2>1.0</mu2>
-		<maxVel>1.0</maxVel>
-		<maxContacts>1</maxContacts>
-		<sensor name="ee_contact_sensor" type="contact">
-			<always_on>true</always_on>
-			<update_rate>250.0</update_rate>
-			<contact>
-				<collision>$(arg prefix)wrist_3_link_collision_collision</collision>
-			</contact>
-		        <plugin name="gazebo_ros_bumper_controller" filename="libgazebo_ros_bumper.so">
-				<bumperTopicName>/ur5/wrench</bumperTopicName>
-				<frameName>$(arg prefix)wrist_3_link</frameName>
-		        	<robotNamespace>ur5</robotNamespace>
-			</plugin>
-		</sensor>
-	</gazebo-->
-    <!--
-      Inject Gazebo ROS Control plugin, which allows us to use ros_control
-      controllers to control the virtual robot hw.
-    -->
+    <!-- Inject Gazebo ROS Control plugin, which allows us to use ros_control controllers to control the virtual robot hw. -->
     <gazebo>
       <plugin name="gazebo_ros_controller_manager" filename="libgazebo_ros_control.so">
